Commit message: joints visible control is bit broken

File: puppyarm/model/PuppyArm.urdf (robot description, URDF)
Before this commit: robot onshape_robot, 45 links, 44 joints
Joints:
- removed joint Part_1_1_2_joint
- removed joint Part_1_1_3_joint
- removed joint Part_1_1_4_joint
- removed joint Part_1_2_2_joint
- removed joint Part_1_2_3_joint
- removed joint Part_1_2_4_joint
- removed joint Part_1_2_joint
- removed joint Part_1_3_2_joint
- removed joint Part_1_3_joint
- removed joint Part_1_8_joint
- removed joint Part_2_2_joint
- removed joint SG_ZIJI_15_1_2_joint
- removed joint SG_ZIJI_15_1_3_joint
- removed joint SG_ZIJI_15_1_4_joint
- removed joint SG_ZIJI_15_1_joint
- removed joint XG_ZIJI_16_1_2_joint
- removed joint XG_ZIJI_16_1_3_joint
- removed joint XG_ZIJI_16_1_4_joint
- removed joint XG_ZIJI_16_1_joint
- removed joint v2_1_3_joint
- removed joint v2_1_7_joint
- added joint Fastened_1: type fixed, parent Part_1_1_2, child Part_2_2, origin xyz=0 0 -0.0085 rpy=0 0 -1.570796
- added joint Fastened_16: type fixed, parent Part_1_3, child Part_1_2, origin xyz=0 0 0.003 rpy=0 0 0
- added joint Fastened_1_2: type fixed, parent SG_ZIJI_15_1_3, child Part_1_3_2, origin xyz=0.0115 -0.0096 -0.00025 rpy=-1.570796 0 1.570796
- added joint Fastened_1_3: type fixed, parent Part_1_2_3, child Part_1_1_3, origin xyz=0 0.0145 -0.0375 rpy=0 0 0
- added joint Fastened_1_4: type fixed, parent Part_1_2_4, child Part_1_1_4, origin xyz=0 -0.0145 -0.035 rpy=-1.570796 0 0
- added joint Fastened_2: type fixed, parent Part_1_1, child Part_1_2_2, origin xyz=0.02565 0 0 rpy=-3.141593 0 0
- added joint Fastened_2_2: type fixed, parent SG_ZIJI_15_1_4, child Part_1_2_3, origin xyz=0.0115 -0.0096 -0.00025 rpy=-1.570796 0 1.570796
- added joint Fastened_3: type fixed, parent v2_1_5, child Part_1_1_2, origin xyz=0.01 0.00875 -0.02 rpy=0 0 -1.570796
- added joint Fastened_4: type fixed, parent Part_1_1_4, child v2_1_7, origin xyz=0.0085 0.073 0.0145 rpy=0 0 1.570796
- added joint Fastened_5: type fixed, parent SG_ZIJI_15_1_2, child Part_1_2_4, origin xyz=0.0115 -0.0096 -0.00025 rpy=-1.570796 0 1.570796
- added joint Fastened_6: type fixed, parent Part_1_2_2, child v2_1_3, origin xyz=0.0085 0.01 0.032 rpy=-3.141593 0 -1.570796
- added joint Fastened_7: type fixed, parent Part_1_8, child Part_1_3, origin xyz=0 0.00075 0.0295 rpy=0 0 0
- added joint Fastened_8: type fixed, parent XG_ZIJI_16_1, child Part_1_8, origin xyz=-0.0255 -0.0316 0 rpy=-1.570796 1.570796 0
- added joint Revolute_1: type revolute, parent v2_1, child SG_ZIJI_15_1, origin xyz=0.03438 0.0177 -0.007473 rpy=0 0.29743 0, axis 0 -1 0
- added joint Revolute_1_2: type revolute, parent v2_1_5, child SG_ZIJI_15_1_3, origin xyz=0.009948 0.0177 0.0255 rpy=-3.141593 -1.568773 -3.141593, axis 0 -1 0
- added joint Revolute_1_3: type revolute, parent v2_1_7, child SG_ZIJI_15_1_4, origin xyz=0.008285 0.0177 -0.025442 rpy=-3.141593 1.5035 3.141593, axis 0 -1 0
- added joint Revolute_1_4: type revolute, parent v2_1_3, child SG_ZIJI_15_1_2, origin xyz=0.03536 0.0177 0.002667 rpy=0 -0.104793 0, axis 0 -1 0
- added joint Revolute_2: type revolute, parent v2_1_2, child XG_ZIJI_16_1, origin xyz=0.019011 -0.04945 -0.023855 rpy=-3.141593 1.209602 0, axis 0 1 0
- added joint Revolute_2_2: type revolute, parent v2_1_6, child XG_ZIJI_16_1_3, origin xyz=0.007532 -0.04945 0.02538 rpy=0 -1.473845 3.141593, axis 0 1 0
- added joint Revolute_2_3: type revolute, parent v2_1_8, child XG_ZIJI_16_1_4, origin xyz=0.012364 -0.04945 -0.02539 rpy=3.141593 1.47795 0, axis 0 1 0
- added joint Revolute_2_4: type revolute, parent v2_1_4, child XG_ZIJI_16_1_2, origin xyz=-0.015077 -0.04945 0.004624 rpy=0 -0.18235 -3.141593, axis 0 1 0
- joint GE_27_1_2_joint: origin xyz=0.087241 0.041018 0.009294 rpy=-1.570796 -0.304321 -2.804608 -> xyz=0.086127 0.06072 0.044993 rpy=-1.570796 -0.069319 -2.681304
- joint GE_27_1_3_joint: origin xyz=-0.049528 -0.014104 -0.093023 rpy=-1.233812 -1.570796 0 -> xyz=-0.049193 -0.013963 -0.093023 rpy=-1.570796 -1.568773 0.460289
- joint GE_27_1_4_joint: origin xyz=-0.05 -0.01427 0.055977 rpy=-1.907781 1.570796 0 -> xyz=-0.049371 -0.014051 0.055978 rpy=1.570796 1.568773 -2.681304
- joint MOTOR_1723_3_1_2_joint: origin xyz=0.070206 0.017195 0.018127 rpy=0 -1.266475 0.336985 -> xyz=0.070899 0.034362 0.048006 rpy=0 -1.501477 0.460289
- joint MOTOR_1723_3_1_3_joint: origin xyz=-0.056279 0.001385 -0.067523 rpy=0 0 -2.804608 -> xyz=-0.057752 0.000601 -0.06752 rpy=0 -0.002023 -2.681304
- joint MOTOR_1723_3_1_4_joint: origin xyz=-0.054392 0.002046 0.030477 rpy=-3.141593 0 0.336985 -> xyz=-0.055782 0.001577 0.030476 rpy=-3.141593 0.002023 0.460289
- joint PCB_CHAZUO_92_1_2_joint: origin xyz=0.062297 0.038636 0.016935 rpy=3.141593 -0.304321 -2.804608 -> xyz=0.060671 0.054795 0.046759 rpy=3.141593 -0.069319 -2.681304
- joint PCB_CHAZUO_92_1_3_joint: origin xyz=-0.047544 -0.019767 -0.067523 rpy=-2.804608 -1.570796 0 -> xyz=-0.046482 -0.019316 -0.067523 rpy=-3.141593 -1.568773 0.460289
- joint PCB_CHAZUO_92_1_4_joint: origin xyz=-0.048016 -0.019932 0.030477 rpy=2.804608 1.570796 0 -> xyz=-0.046752 -0.01945 0.030478 rpy=0 1.568773 -2.681304
- joint Part_1_1_joint: origin xyz=0.079209 0.061992 -0.0227 rpy=3.121406 0 -1.233812 -> xyz=0.071188 0.078371 0.013477 rpy=2.96748 0 -1.110507
- joint ZK_122_1_2_joint: origin xyz=0.062297 0.038636 0.016935 rpy=3.141593 -0.304321 -2.804608 -> xyz=0.060671 0.054795 0.046759 rpy=3.141593 -0.069319 -2.681304
- joint ZK_122_1_3_joint: origin xyz=-0.047544 -0.019767 -0.067523 rpy=-2.804608 -1.570796 0 -> xyz=-0.046482 -0.019316 -0.067523 rpy=-3.141593 -1.568773 0.460289
- joint ZK_122_1_4_joint: origin xyz=-0.048016 -0.019932 0.030477 rpy=2.804608 1.570796 0 -> xyz=-0.046752 -0.01945 0.030478 rpy=0 1.568773 -2.681304
- joint v2_1_4_joint: origin xyz=0.092467 -0.003191 0.011784 rpy=-3.141593 0.251669 0.336985 -> xyz=0.096751 0.01749 0.047483 rpy=-3.141593 0.251669 0.460289
- joint v2_1_5_joint: origin xyz=-0.043959 0.000244 -0.093023 rpy=0 0 -2.804608 -> xyz=-0.045431 0.000961 -0.093023 rpy=0 0 -2.681304
- joint v2_1_6_joint: origin xyz=-0.073286 0.023612 -0.092034 rpy=0 0.098974 0.336985 -> xyz=-0.07741 0.020544 -0.092034 rpy=0 0.098974 0.460289
- joint v2_1_8_joint: origin xyz=-0.073762 0.023445 0.056925 rpy=0 0.09487 0.336985 -> xyz=-0.077591 0.020454 0.056925 rpy=0 0.09487 0.460289
